Commit message: rgbd sensor added

File: create_autonomy-indigo-devel/ca_description/urdf/create_base.urdf.xacro (robot description, xacro)
@@ -132,5 +132,5 @@
     <xacro:create_wheel prefix="left" y_offset="${wheel_separation / 2}" wheel_radius="${wheel_radius}" wheel_width="${wheel_width}"/>
     <xacro:create_wheel prefix="right" y_offset="${wheel_separation / -2}" wheel_radius="${wheel_radius}" wheel_width="${wheel_width}"/>
-    <!--<link name="rear_wheel_link">
+    <link name="rear_wheel_link">
     <inertial>
       <origin xyz="0 0 0"/>
@@ -142,11 +142,11 @@
       <origin xyz="0 0 0" rpy="0 ${PI/2} ${PI/2}"/>
       <geometry>
-        <sphere radius="0.015" />
-      </geometry>
-    </visual>
-    <collision>
-      <origin xyz="0 0 0" rpy="0 ${PI/2} ${PI/2}" />
-      <geometry>
-        <sphere radius="0.015" />
+        <sphere radius="0.021" />
+      </geometry>
+    </visual>
+    <collision>
+      <origin xyz="0 0 0" rpy="0 ${PI/2} ${PI/2}" />
+      <geometry>
+        <sphere radius="0.021" />
       </geometry>
     </collision>
@@ -157,5 +157,5 @@
       <child link="rear_wheel_link"/>
       <axis xyz="0 1 0"/>
-    </joint>-->
+    </joint>
     <link name="front_wheel_link">
     <inertial>
@@ -167,11 +167,11 @@
       <origin xyz="0 0 0" rpy="0 ${PI/2} ${PI/2}" />
       <geometry>
-        <sphere radius="0.018" />
-      </geometry>
-    </visual>
-    <collision>
-      <origin xyz="0 0 0" rpy="0 ${PI/2} ${PI/2}" />
-      <geometry>
-        <sphere radius="0.018" />
+        <sphere radius="0.021" />
+      </geometry>
+    </visual>
+    <collision>
+      <origin xyz="0 0 0" rpy="0 ${PI/2} ${PI/2}" />
+      <geometry>
+        <sphere radius="0.021" />
       </geometry>
     </collision>
@@ -221,4 +221,96 @@
     </inertial>
    </link>
+   <link name="yaw_platform">
+    <inertial>
+      <mass value="1e-5" />
+      <origin xyz="0 0 0" rpy="0 0 0"/>
+      <inertia ixx="1e-6" ixy="0" ixz="0" iyy="1e-6" iyz="0" izz="1e-6" />
+    </inertial>
+    <visual>
+      <origin xyz="0 0 0" rpy="0 0 1.57079632" />
+      <geometry>
+        <mesh filename="package://robot_sim_demo/models/meshes/yaw_platform.dae" />
+      </geometry>
+    </visual>
+    <collision>
+      <origin xyz="0 0 0" rpy="0 0 1.57079632" />
+      <geometry>
+        <box size="0.1 0.1 0.1"/>
+      </geometry>
+    </collision>
+  </link>
+  <joint name="base_to_yaw_platform" type="revolute">
+    <axis xyz="0 0 1"/>
+    <parent link="base_link"/>
+    <child link="yaw_platform"/>
+    <origin rpy="0 0 0" xyz="0 0 1.305"/>
+    <limit effort="100" velocity="100" lower="-1.57" upper="1.57" />
+    <dynamics damping="0.0" friction="10.0"/>
+  </joint>
+  <link name="pitch_platform">
+    <inertial>
+      <mass value="1e-5" />
+      <origin xyz="0 0 0" rpy="0 0 0"/>
+      <inertia ixx="1e-6" ixy="0" ixz="0" iyy="1e-6" iyz="0" izz="1e-6" />
+    </inertial>
+    <visual>
+      <origin xyz="0 0 0" rpy="0 0 0" />
+      <geometry>
+        <mesh filename="package://robot_sim_demo/models/meshes/pitch_platform.dae" />
+      </geometry>
+    </visual>
+    <collision>
+      <origin xyz="0 0 0" rpy="0 0 0" />
+      <geometry>
+        <box size="0.1 0.1 0.1"/>
+      </geometry>
+    </collision>
+  </link>
+  <joint name="yaw_to_pitch_platform" type="revolute">
+    <axis xyz="0 1 0"/>
+    <parent link="yaw_platform"/>
+    <child link="pitch_platform"/>
+    <origin rpy="0 0 0" xyz="0 0 0"/>
+    <limit effort="100" velocity="100" lower="-1.57" upper="1.57" />
+    <dynamics damping="0.0" friction="10.0"/>
+  </joint>
+  <!-- Camera -->
+  <link name="camera_link">
+    <collision>
+      <origin xyz="0 0 0" rpy="0 0 0"/>
+      <geometry>
+        <box size="0.1 0.1 0.1"/>
+      </geometry>
+    </collision>
+    <visual>
+      <origin xyz="0 0 0" rpy="0 0 0"/>
+      <geometry>
+        <!--<mesh filename="package://robot_sim_demo/models/meshes/xtion_pro_camera.dae" />-->
+        <mesh filename="package://robot_sim_demo/models/meshes/realsense.dae" />
+      </geometry>
+    </visual>
+    <inertial>
+      <mass value="1e-5" />
+      <origin xyz="0 0 0" rpy="0 0 0"/>
+      <inertia ixx="1e-6" ixy="0" ixz="0" iyy="1e-6" iyz="0" izz="1e-6" />
+    </inertial>
+  </link>
+  <joint name="camera_joint" type="fixed">
+    <axis xyz="0 1 0" />
+    <origin xyz="-0.005 0 .06" rpy="0 0 0"/>
+    <parent link="pitch_platform"/>
+    <child link="camera_link"/>
+  </joint>
+  <!-- generate an optical frame http://www.ros.org/reps/rep-0103.html#suffix-frames
+      so that ros and opencv can operate on the camera frame correctly -->
+  <joint name="camera_optical_joint" type="fixed">
+    <!-- these values have to be these values otherwise the gazebo camera image
+        won't be aligned properly with the frame it is supposedly originating from -->
+    <origin xyz="0 0 0" rpy="-1.5708 0 -1.5708"/>
+    <parent link="camera_link"/>
+    <child link="camera_link_optical"/>
+  </joint>
+  <link name="camera_link_optical">
+  </link>
     <!-- Simulation sensors -->
     <xacro:sim_create_base/>

File: create_autonomy-indigo-devel/ca_description/urdf/create_base_gazebo.urdf.xacro (robot description, xacro)
@@ -230,4 +230,27 @@
     </sensor>
   </gazebo>
+    <!-- camera -->
+    <gazebo reference="camera_link">
+      <sensor type="depth" name="camera">
+        <plugin name="kinect_camera_controller" filename="libgazebo_ros_openni_kinect.so">
+          <cameraName>camera</cameraName>
+          <alwaysOn>true</alwaysOn>
+          <updateRate>10</updateRate>
+          <imageTopicName>rgb/image_raw</imageTopicName>
+          <depthImageTopicName>depth/image_raw</depthImageTopicName>
+          <pointCloudTopicName>depth/points</pointCloudTopicName>
+          <cameraInfoTopicName>rgb/camera_info</cameraInfoTopicName>
+          <depthImageCameraInfoTopicName>depth/camera_info</depthImageCameraInfoTopicName>
+          <frameName>camera_link_optical</frameName>
+          <baseline>0.1</baseline>
+          <distortion_k1>0.0</distortion_k1>
+          <distortion_k2>0.0</distortion_k2>
+          <distortion_k3>0.0</distortion_k3>
+          <distortion_t1>0.0</distortion_t1>
+          <distortion_t2>0.0</distortion_t2>
+          <pointCloudCutoff>0.4</pointCloudCutoff>
+        </plugin>
+      </sensor>
+    </gazebo>
   </xacro:macro>
 </robot>

Commit message: ROS.md update

File: create_autonomy-indigo-devel/ca_description/urdf/create_base.urdf.xacro (robot description, xacro)
@@ -142,11 +142,11 @@
       <origin xyz="0 0 0" rpy="0 ${PI/2} ${PI/2}"/>
       <geometry>
-        <sphere radius="0.021" />
-      </geometry>
-    </visual>
-    <collision>
-      <origin xyz="0 0 0" rpy="0 ${PI/2} ${PI/2}" />
-      <geometry>
-        <sphere radius="0.021" />
+        <sphere radius="0.020" />
+      </geometry>
+    </visual>
+    <collision>
+      <origin xyz="0 0 0" rpy="0 ${PI/2} ${PI/2}" />
+      <geometry>
+        <sphere radius="0.020" />
       </geometry>
     </collision>
@@ -167,11 +167,11 @@
       <origin xyz="0 0 0" rpy="0 ${PI/2} ${PI/2}" />
       <geometry>
-        <sphere radius="0.021" />
-      </geometry>
-    </visual>
-    <collision>
-      <origin xyz="0 0 0" rpy="0 ${PI/2} ${PI/2}" />
-      <geometry>
-        <sphere radius="0.021" />
+        <sphere radius="0.020" />
+      </geometry>
+    </visual>
+    <collision>
+      <origin xyz="0 0 0" rpy="0 ${PI/2} ${PI/2}" />
+      <geometry>
+        <sphere radius="0.020" />
       </geometry>
     </collision>

Commit message: move-base reconfiguration

File: create_autonomy-indigo-devel/ca_description/urdf/create_base.urdf.xacro (robot description, xacro)
@@ -221,5 +221,5 @@
     </inertial>
    </link>
-   <link name="yaw_platform">
+   <link name="platform">
     <inertial>
       <mass value="1e-5" />
@@ -230,48 +230,18 @@
       <origin xyz="0 0 0" rpy="0 0 1.57079632" />
       <geometry>
-        <mesh filename="package://robot_sim_demo/models/meshes/yaw_platform.dae" />
-      </geometry>
-    </visual>
-    <collision>
-      <origin xyz="0 0 0" rpy="0 0 1.57079632" />
-      <geometry>
         <box size="0.1 0.1 0.1"/>
       </geometry>
+    </visual>
+    <collision>
+      <origin xyz="0 0 0" rpy="0 0 0" />
+      <geometry>
+        <box size="0.1 0.1 0.1"/>
+      </geometry>
     </collision>
   </link>
-  <joint name="base_to_yaw_platform" type="revolute">
-    <axis xyz="0 0 1"/>
+  <joint name="base_to_platform" type="fixed">
     <parent link="base_link"/>
-    <child link="yaw_platform"/>
-    <origin rpy="0 0 0" xyz="0 0 1.305"/>
-    <limit effort="100" velocity="100" lower="-1.57" upper="1.57" />
-    <dynamics damping="0.0" friction="10.0"/>
-  </joint>
-  <link name="pitch_platform">
-    <inertial>
-      <mass value="1e-5" />
-      <origin xyz="0 0 0" rpy="0 0 0"/>
-      <inertia ixx="1e-6" ixy="0" ixz="0" iyy="1e-6" iyz="0" izz="1e-6" />
-    </inertial>
-    <visual>
-      <origin xyz="0 0 0" rpy="0 0 0" />
-      <geometry>
-        <mesh filename="package://robot_sim_demo/models/meshes/pitch_platform.dae" />
-      </geometry>
-    </visual>
-    <collision>
-      <origin xyz="0 0 0" rpy="0 0 0" />
-      <geometry>
-        <box size="0.1 0.1 0.1"/>
-      </geometry>
-    </collision>
-  </link>
-  <joint name="yaw_to_pitch_platform" type="revolute">
-    <axis xyz="0 1 0"/>
-    <parent link="yaw_platform"/>
-    <child link="pitch_platform"/>
-    <origin rpy="0 0 0" xyz="0 0 0"/>
-    <limit effort="100" velocity="100" lower="-1.57" upper="1.57" />
-    <dynamics damping="0.0" friction="10.0"/>
+    <child link="platform"/>
+    <origin rpy="0 0 0" xyz="0 0 0.3"/>
   </joint>
   <!-- Camera -->
@@ -297,7 +267,6 @@
   </link>
   <joint name="camera_joint" type="fixed">
-    <axis xyz="0 1 0" />
     <origin xyz="-0.005 0 .06" rpy="0 0 0"/>
-    <parent link="pitch_platform"/>
+    <parent link="platform"/>
     <child link="camera_link"/>
   </joint>

Commit message: base_laser_link tf_fix

File: create_autonomy-indigo-devel/ca_description/urdf/create_base.urdf.xacro (robot description, xacro)
@@ -198,5 +198,5 @@
     </link>
     <joint name="laser_joint" type="fixed">
-    <origin xyz=".115 0 0.12" rpy="0 0 0" />
+    <origin xyz="0.04 0 0.12" rpy="0 0 0" />
     <parent link="base_link" />
     <child link="base_laser_link" />
